File: pcb/ykb.kicad_pcb (KiCad board)
At the start: 2 copper layers, 299.2 x 132.3 mm, 90 parts, among them J1 Conn_01x07_Socket, U1 Helios

Commit message: ideally, finalised routing
Parts:
- moved D14 11.1 mm to (185.9, 162.1)
- moved D19 11.1 mm to (207.8, 192.9)
- moved D26 11.1 mm to (362.8, 154.2)
- moved D27 11.1 mm to (359.6, 137.5)
- moved D29 11.1 mm to (342.2, 146.6)
- moved S13 11.1 mm to (171.9, 166.8)
- moved S16 11.1 mm to (184.5, 180.2)
- moved S17 11.1 mm to (194.5, 166.4)
- moved S26 11.1 mm to (353.4, 150.6)
- moved S35 11.1 mm to (301.7, 166.8)
- moved D2 11.1 mm to (110.8, 141.7)
- moved D12 11.1 mm to (182.8, 129.4)
- moved D28 11.1 mm to (356.3, 120.9)
- moved D34 11.1 mm to (305.8, 121.1)
- moved S3 11.1 mm to (104.6, 119.0)
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Routing:
- net row 1: track 446.0 -> 446.7 mm

Commit message: teardrops on pads
Routing:
- net DCS: track 18.2 -> 18.5 mm, vias 1 -> 0
- net DRST: vias 1 -> 0

Commit message: plate started, standoff holes placed
Parts:
- added ?: , , F.Cu at (173.8, 206.1)
- added ?: , , B.Cu at (356.8, 108.6)
- added ?: , , F.Cu at (216.8, 158.6)
- added ?: , , F.Cu at (116.8, 108.6)
- added ?: , , F.Cu at (111.8, 165.1)
- added ?: , , F.Cu at (190.3, 124.6)
- added ?: , , B.Cu at (361.8, 165.1)
- added ?: , , B.Cu at (299.8, 206.1)
- added ?: , , B.Cu at (256.8, 158.6)
- added ?: , , B.Cu at (283.3, 124.6)

Commit message: done
Parts:
- S1, S10, S11, S12, S13, S14, S15, S16, S17, S18, S19, S2, S20, S21, S22, S23, S24, S25, S26, S27, S28, S29, S3, S30, S31, S32, S33, S34, S35, S36, S37, S38, S39, S4, S40, S41, S42, S43, S44, S5, S6, S7, S8, S9: footprint ScottoKeebs_Hotswap:Hotswap_Choc_V1V2_1.00u -> keyswitches:Kailh_socket_PG1350_optional
- moved S25 15.0 mm to (369.0, 104.1)
- moved D18 15.0 mm to (208.3, 147.0)
- moved D1 15.0 mm to (109.0, 143.7)
- moved D2 15.0 mm to (110.8, 126.7)
- moved S34 15.0 mm to (295.7, 105.9)
- moved D30 15.0 mm to (334.7, 116.2)
- moved S27 15.0 mm to (350.2, 119.0)
- moved S17 15.0 mm to (194.5, 151.5)
- moved S21 15.0 mm to (166.9, 181.8)
- moved D17 15.0 mm to (198.2, 160.9)
- moved D32 15.0 mm to (323.2, 135.2)
- moved S8 15.0 mm to (148.9, 115.2)
- moved S39 15.0 mm to (279.2, 151.5)
- moved U1 15.0 mm to (236.8, 151.0)
- moved S18 15.0 mm to (204.5, 137.7)
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Routing:
- net col 9: track 271.2 -> 314.3 mm
- net col 2: track 270.0 -> 312.5 mm
- net col 3: track 252.8 -> 292.3 mm
- net col 8: track 256.2 -> 294.9 mm
- net col 7: track 229.9 -> 264.2 mm
- net col 4: track 237.4 -> 269.1 mm
- net col 6: track 194.7 -> 225.0 mm
- net col 1: track 261.1 -> 286.9 mm
- net col 10: track 255.8 -> 281.7 mm
- net col 5: track 208.3 -> 227.8 mm
- net col 0: track 271.8 -> 288.8 mm
- net col 11: track 271.5 -> 288.4 mm
- net Net-(D26-A): track 7.64 -> 21.9 mm, vias 0 -> 1
- net Net-(D20-A): track 7.35 -> 21.4 mm, vias 0 -> 1
- net Net-(D11-A): track 6.92 -> 20.7 mm, vias 0 -> 1
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